File: Rocket Igniter SMT/Rocket Igniter SMT.sch (KiCad schematic (older format))
At the start: 25 parts, among them J1 1711725, J2 1711725, K1 G5Q-1 DC5, Q1 BC327, Q2 PN2222ABU, SW1 M2011S3S1W01, SW2 RP3502ARED, SW3 Y201132C203NQ

Commit message: checkpoint
Parts:
- C1: value 35PX680MEFC10X16 -> 560µF; footprint Capacitor_THT:C_Radial_D10.0mm_H16.0mm_P5.00mm -> Capacitor_SMD:CP_Elec_10x10; Manufacturer Part (none) -> VZS561M1ETR-1010; Part 35PX680MEFC10X16 -> C249979; Spice_Model 680u -> 560uF
- C2, C3: value 860010572002 -> 10µF; footprint Capacitor_THT:C_Radial_D5.0mm_H11.0mm_P2.00mm -> Capacitor_SMD:C_0603_1608Metric; Manufacturer Part (none) -> CL10A106KP8NNNC; Part 860010572002 -> C19702; Spice_Model (none) -> 10uF; Spice_Netlist_Enabled (none) -> Y; Spice_Primitive (none) -> C
- D1: value 1N5819-E3/54 -> B5819W SL; footprint Diode_THT:D_DO-41_SOD81_P10.16mm_Horizontal -> Diode_SMD:D_SOD-123; Manufacturer Part (none) -> B5819W SL; Part 1N5819-E3/54 -> C8598; Spice_Model 1N5819-E3/54 -> (none)
- D2: value 1N6267A-E3/54 -> SMFJ7.0CA; footprint Diode_THT:D_DO-15_P10.16mm_Horizontal -> Diode_SMD:D_SOD-123F; Manufacturer Part (none) -> SMFJ7.0CA; Part 1N6267A-E3/54 -> C511920; Spice_Netlist_Enabled (none) -> Y; Spice_Primitive (none) -> D
- J1, J2: DigiKey Part (none) -> 277-1027-ND; Manufacturer Part (none) -> 1711725; Part 1711725 -> (none)
- K1: DigiKey Part (none) -> Z12713-ND; Manufacturer Part (none) -> G5Q-1 DC5; Part G5Q-1 DC5 -> (none)
- LED1: DigiKey Part (none) -> 350-2797-ND; Part 5592201003F -> (none)
- LED2: DigiKey Part (none) -> 350-2799-ND; Part 5592301003F -> (none)
- LED3: DigiKey Part (none) -> 350-2796-ND; Part 5592101003F -> (none)
- Q1: DigiKey Part (none) -> 2156-BC327-FS-ND; Manufacturer Part (none) -> BC327; Part BC327 -> (none)
- Q2: value PN2222ABU -> S8050 J3Y; footprint Package_TO_SOT_THT:TO-92_Inline -> Package_TO_SOT_SMD:SOT-23; Manufacturer Part (none) -> S8050 J3Y; Part PN2222ABU -> C2146
- R1: value 33k -> 33kΩ; footprint Resistor_THT:R_Axial_DIN0207_L6.3mm_D2.5mm_P10.16mm_Horizontal -> Resistor_SMD:R_0603_1608Metric; Part (none) -> C4216
- R2, R4, R7: value 220 -> 220Ω; footprint Resistor_THT:R_Axial_DIN0207_L6.3mm_D2.5mm_P10.16mm_Horizontal -> Resistor_SMD:R_0603_1608Metric; Part (none) -> C22962; Spice_Model (none) -> 220; Spice_Netlist_Enabled (none) -> Y; Spice_Primitive (none) -> R
- R3, R5, R6: value 33k -> 33kΩ; footprint Resistor_THT:R_Axial_DIN0207_L6.3mm_D2.5mm_P10.16mm_Horizontal -> Resistor_SMD:R_0603_1608Metric; Part (none) -> C4216; Spice_Model (none) -> 33k; Spice_Netlist_Enabled (none) -> Y; Spice_Primitive (none) -> R
- R8: value 1k -> 1kΩ; footprint Resistor_THT:R_Axial_DIN0207_L6.3mm_D2.5mm_P10.16mm_Horizontal -> Resistor_SMD:R_0603_1608Metric; Part (none) -> C21190; Spice_Model (none) -> 1k; Spice_Netlist_Enabled (none) -> Y; Spice_Primitive (none) -> R
- SW1: DigiKey Part (none) -> 360-3695-ND; Manufacturer Part (none) -> M2011S3S1W01; Part M2011S3S1W01 -> (none)
- SW2: DigiKey Part (none) -> EG1930-ND; Manufacturer Part (none) -> RP3502ARED; Part RP3502ARED -> (none)
- SW3: DigiKey Part (none) -> CKN11519-ND; Manufacturer Part (none) -> Y201132C203NQ; Part Y201132C203NQ -> (none)
- VR1: DigiKey Part (none) -> AS7805AT-E1DI-ND; Manufacturer Part (none) -> AS7805AT-E1; Part AS7805AT-E1 -> (none)
